File: PCB/Charging_PCB_v102/charge_pcb.kicad_pcb (KiCad board)
At the start: 2 copper layers, 96.5 x 50.8 mm, 40 parts, among them J1 PCB_1, J2 Battery, J3 Power Switch, J4 24V Out, J5 Motor_Drive, J6 Motor_Cutter, J7 24V Out, J8 Start, J9 24V out, Q1 BC547C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

Commit message: PCB
Routing:
- net Net-(D2-Pad2): track 30.1 -> 50.9 mm
- net Net-(D3-Pad1): track 32.5 -> 52.8 mm
Other:
- board text added: "PowerBoard by S.D/B.B V1.02"
- board text removed: "PowerBoard by S.D/B.B V1.01"
