File: PCB/Power_PCB_v105/charge_pcb.kicad_pcb (KiCad board)
At the start: 2 copper layers, 129.5 x 66 mm, 48 parts, among them J1 Main_PCB2, J10 Mot_Left, J11 DC/DC1, J12 DC/DC2, J2 Battery, J3 Power Switch, J4 Mow3, J5 Main_PCB1, J6 Mow2, J7 Mow1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

Commit message: power route
Parts:
- J10 M Left +: renamed from J10
- J11 DC/DC1: renamed from J11
- J12 DC/DC2: renamed from J12
- J2 BAT: renamed from J2
- J3 SWITCH: renamed from J3
- J4 Mow3 +: renamed from J4
- J6 Mow2 +: renamed from J6
- J7 Mow1 +: renamed from J7
- J9 M Right +: renamed from J9
- U1 CHARGE CURRENT: renamed from U1
- U2 Mot Left Current: renamed from U2
- U3 Mow3 Current: renamed from U3
- U4 Mow2 Current: renamed from U4
- U5 Mow1 Current: renamed from U5
- U6 Mot Right Current: renamed from U6
- moved R6 82.8 mm to (143.1, 90.4)
- moved R4 49.6 mm to (102.0, 106.3)
- moved R3 49.4 mm to (102.0, 102.9)
- moved R11 49.0 mm to (94.4, 99.4)
- moved D4 48.8 mm to (151.9, 85.2), turned to 90 degrees
- moved J2 BAT 47.1 mm to (205.7, 105.3)
- moved J3 SWITCH 47.1 mm to (205.6, 93.1)
- moved J8 45.5 mm to (154.7, 68.1)
- moved F2 45.3 mm to (166.8, 76.8)
- moved R10 44.9 mm to (94.4, 96.1)
- moved R9 44.9 mm to (114.6, 77.5)
- moved H3 44.8 mm to (209.2, 118.2)
- moved H4 44.8 mm to (89.3, 118.2)
- moved Q2 44.8 mm to (114.7, 87.2)
- moved H2 44.8 mm to (209.2, 64.9)
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Routing:
- net GND: track 0.00 -> 522.1 mm
- net V_Bat: track 0.00 -> 214.1 mm
- net +3V3: track 0.00 -> 146.2 mm
- net SCL0: track 0.00 -> 131.5 mm
- net SDA0: track 0.00 -> 127.8 mm, vias 0 -> 1
- net Net-(J2-Pad1): track 0.00 -> 111.8 mm
- net SCL1: track 0.00 -> 76.8 mm
- net SDA1: track 0.00 -> 76.5 mm
- net Net-(F2-Pad1): track 0.00 -> 63.5 mm
- net Net-(Q3-Pad2): track 0.00 -> 58.5 mm
- net V_Charge: track 0.00 -> 50.8 mm
- net Net-(D5-Pad2): track 0.00 -> 50.8 mm
- net Net-(D2-Pad2): track 0.00 -> 42.4 mm
- net Net-(Q1-Pad1): track 0.00 -> 39.9 mm
- net Net-(D11-Pad2): track 0.00 -> 37.7 mm
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Other:
- board size 129.5 x 66 mm -> 128.1 x 64 mm
- board text added: "++"
- board text added: "--"
- board text added: "Power Board V1.05"
- board text removed: "PowerBoard V1.05"

Commit message: teensy pcb
Routing:
- net GND: track 522.1 -> 593.1 mm
Other:
- board text removed: "3.3V"
- board text removed: "BatterySwitch"
- board text removed: "BatteryVoltage"
- board text removed: "ChargeCurrent"
- board text removed: "ChargeEnable"
- board text removed: "ChargeVoltage"
Changed lines of the file:
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@@
   (general
     (thickness 1.6)
-    (drawings 24)
-    (tracks 371)
+    (drawings 10)
+    (tracks 375)
     (zones 0)
     (modules 48)
@@
     (34 B.Paste user)
     (35 F.Paste user)
-    (36 B.SilkS user hide)
+    (36 B.SilkS user)
     (37 F.SilkS user)
     (38 B.Mask user)
@@
   )
   (setup
-    (last_trace_width 1.25)
+    (last_trace_width 2)
     (user_trace_width 0.4)
     (user_trace_width 0.5)
@@
     (effects (font (size 1 1) (thickness 0.15)) (justify mirror))
   )
-  (gr_text + (at 148.59 147.32) (layer B.SilkS)
-    (effects (font (size 1 1) (thickness 0.15)) (justify mirror))
-  )
-  (gr_text + (at 137.16 147.32) (layer B.SilkS)
-    (effects (font (size 1 1) (thickness 0.15)) (justify mirror))
-  )
-  (gr_text + (at 125.73 147.32) (layer B.SilkS)
-    (effects (font (size 1 1) (thickness 0.15)) (justify mirror))
-  )
-  (gr_text + (at 78.74 114.3) (layer B.SilkS)
-    (effects (font (size 1 1) (thickness 0.15)) (justify mirror))
-  )
-  (gr_text GND (at 78.74 119.38 90) (layer B.SilkS)
-    (effects (font (size 1 1) (thickness 0.15)) (justify mirror))
-  )
-  (gr_text GND (at 153.67 147.32) (layer B.SilkS)
-    (effects (font (size 1 1) (thickness 0.15)) (justify mirror))
-  )
-  (gr_text GND (at 142.24 147.32) (layer B.SilkS)
-    (effects (font (size 1 1) (thickness 0.15)) (justify mirror))
-  )
-  (gr_text GND (at 130.81 147.32) (layer B.SilkS)
-    (effects (font (size 1 1) (thickness 0.15)) (justify mirror))
-  )
   (gr_text GND (at 134.62 111.76) (layer B.SilkS)
     (effects (font (size 1 1) (thickness 0.15)) (justify mirror))
@@
   (gr_text "Power\nBoard\nV1.05" (at 98.425 115.189) (layer F.SilkS)
     (effects (font (size 1.5 1.5) (thickness 0.3)))
-  )
-  (gr_text BatteryVoltage (at 75.05 141.6) (layer B.SilkS)
-    (effects (font (size 1 1) (thickness 0.25)) (justify mirror))
-  )
-  (gr_text BatterySwitch (at 75.4 138.94) (layer B.SilkS)
-    (effects (font (size 1 1) (thickness 0.25)) (justify mirror))
-  )
-  (gr_text ChargeVoltage (at 75.05 136.46) (layer B.SilkS)
-    (effects (font (size 1 1) (thickness 0.25)) (justify mirror))
-  )
-  (gr_text ChargeCurrent (at 74.87 133.89) (layer B.SilkS)
-    (effects (font (size 1 1) (thickness 0.25)) (justify mirror))
-  )
-  (gr_text ChargeEnable (at 75.22 131.41) (layer B.SilkS)
-    (effects (font (size 1 1) (thickness 0.25)) (justify mirror))
-  )
-  (gr_text 3.3V (at 78.74 128.93) (layer B.SilkS)
-    (effects (font (size 1 1) (thickness 0.25)) (justify mirror))
   )
   (gr_line (start 212.852 61.217) (end 84.709 61.217) (layer Edge.Cuts) (width 0.15))
@@
   (gr_line (start 84.709 125.217) (end 212.852 125.217) (layer Edge.Cuts) (width 0.15))
   (gr_line (start 84.709 61.217) (end 84.709 125.217) (layer Edge.Cuts) (width 0.15))
-  (segment (start 117.6777 82.267) (end 116.5364 81.1257) (width 0.254) (layer F.Cu) (net 1))
-  (segment (start 116.5364 81.1257) (end 109.0616 81.1257) (width 0.254) (layer F.Cu) (net 1))
-  (segment (start 109.0616 81.1257) (end 107.8803 82.307) (width 0.254) (layer F.Cu) (net 1))
   (segment (start 149.5139 80.8879) (end 149.5139 90.8747) (width 0.254) (layer B.Cu) (net 1))
   (segment (start 149.5139 90.8747) (end 150.6059 91.9667) (width 0.254) (layer B.Cu) (net 1))
@@
   (segment (start 88.392 88.171) (end 90.8563 88.171) (width 0.254) (layer B.Cu) (net 1))
   (segment (start 90.8563 88.171) (end 95.459 83.5683) (width 0.254) (layer B.Cu) (net 1))
-  (segment (start 118.959 82.267) (end 117.6777 82.267) (width 0.254) (layer F.Cu) (net 1))
-  (segment (start 106.699 82.307) (end 107.8803 82.307) (width 0.254) (layer F.Cu) (net 1))
   (segment (start 110.109 94.488) (end 108.458 96.139) (width 0.254) (layer F.Cu) (net 1))
   (segment (start 108.458 96.139) (end 101.981 96.139) (width 0.254) (layer F.Cu) (net 1))
@@
   (segment (start 91.769 78.497) (end 95.459 82.187) (width 2) (layer B.Cu) (net 1))
   (segment (start 91.769 77.647) (end 91.769 78.497) (width 2) (layer B.Cu) (net 1))
-  (segment (start 89.475 88.171) (end 88.392 88.171) (width 2) (layer B.Cu) (net 1))
-  (segment (start 95.459 82.187) (end 89.475 88.171) (width 2) (layer B.Cu) (net 1))
   (segment (start 101.339 88.067) (end 101.339 89.027) (width 2) (layer B.Cu) (net 1))
   (segment (start 95.459 82.187) (end 101.339 88.067) (width 2) (layer B.Cu) (net 1))
@@
   (segment (start 198.247 81.026) (end 200.025 79.248) (width 2) (layer F.Cu) (net 1))
   (segment (start 176.403 81.026) (end 198.247 81.026) (width 2) (layer F.Cu) (net 1))
+  (segment (start 116.944999 80.252999) (end 118.959 82.267) (width 2) (layer F.Cu) (net 1))
+  (segment (start 108.753001 80.252999) (end 116.944999 80.252999) (width 2) (layer F.Cu) (net 1))
+  (segment (start 106.699 82.307) (end 108.753001 80.252999) (width 2) (layer F.Cu) (net 1))
+  (segment (start 153.447999 119.284999) (end 154.305 120.142) (width 2) (layer B.Cu) (net 1))
+  (segment (start 141.408029 119.284999) (end 153.447999 119.284999) (width 2) (layer B.Cu) (net 1))
+  (segment (start 139.511029 117.387999) (end 141.408029 119.284999) (width 2) (layer B.Cu) (net 1))
+  (segment (start 134.072001 117.387999) (end 139.511029 117.387999) (width 2) (layer B.Cu) (net 1))
+  (segment (start 131.318 120.142) (end 134.072001 117.387999) (width 2) (layer B.Cu) (net 1))
+  (segment (start 210.621011 116.784989) (end 209.169 118.237) (width 2) (layer B.Cu) (net 1))
+  (segment (start 210.621011 66.349011) (end 210.621011 116.784989) (width 2) (layer B.Cu) (net 1))
+  (segment (start 209.169 64.897) (end 210.621011 66.349011) (width 2) (layer B.Cu) (net 1))
   (segment (start 98.7483 69.167) (end 98.7483 70.798) (width 0.254) (layer B.Cu) (net 2))
   (segment (start 91.769 72.567) (end 96.9793 72.567) (width 2) (layer B.Cu) (net 2))
