File: PCB/TEENSY_PCB_V1.00/Ardumower.sch (KiCad schematic (older format))
At the start: 38 parts, among them J10 Sonar_R, J12 Sonar_L, J13 P_Right, J14 Buzzer, J15 Button, J19 P_Left, J2 I2C2, J21 PCB_2, J23 Ser1, J25 5V IN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

Commit message: gy521 test
Parts:
- JP1: renamed from JP?; footprint (none) -> Connector_PinSocket_2.54mm:PinSocket_1x03_P2.54mm_Vertical
- U1: symbol doit-esp32-devkit-v1:DOIT-ESP32-DEVKIT-V1 -> Ardumower-rescue:DOIT-ESP32-DEVKIT-V1-doit-esp32-devkit-v1
Connections:
- wire segments 41 -> 45
- no-connect marks 3 -> 18
Other:
- moved on the sheet: JP1
Changed lines of the file:
@@
 NoConn ~ 11180 5820
 $Comp
-L doit-esp32-devkit-v1:DOIT-ESP32-DEVKIT-V1 U1
+L Ardumower-rescue:DOIT-ESP32-DEVKIT-V1-doit-esp32-devkit-v1 U1
 U 1 1 60E66356
 P 7870 1985
@@
 L power:+5V #PWR09
 U 1 1 60E9FFBD
-P 6920 3385
-F 0 "#PWR09" H 6920 3235 50  0001 C CNN
-F 1 "+5V" H 6935 3558 50  0000 C CNN
-F 2 "" H 6920 3385 50  0001 C CNN
-F 3 "" H 6920 3385 50  0001 C CNN
-	1    6920 3385
+P 6817 3442
+F 0 "#PWR09" H 6817 3292 50  0001 C CNN
+F 1 "+5V" H 6832 3615 50  0000 C CNN
+F 2 "" H 6817 3442 50  0001 C CNN
+F 3 "" H 6817 3442 50  0001 C CNN
+	1    6817 3442
 	0    -1   -1   0
 $EndComp
@@
 TX1
 Wire Wire Line
-	5695 840  5845 840
+	4480 860  4250 860
+Wire Wire Line
+	4250 860  4250 850
 $Comp
 L power:+3.3V #PWR050
 U 1 1 60C9BB63
-P 5845 840
-F 0 "#PWR050" H 5845 690 50  0001 C CNN
-F 1 "+3.3V" H 5860 1013 50  0000 C CNN
-F 2 "" H 5845 840 50  0001 C CNN
-F 3 "" H 5845 840 50  0001 C CNN
-	1    5845 840
-	0    1    1    0
-$EndComp
-Wire Wire Line
-	4480 860  4250 860
-Wire Wire Line
-	4250 860  4250 850
+P 5290 960
+F 0 "#PWR050" H 5290 810 50  0001 C CNN
+F 1 "+3.3V" H 5305 1133 50  0000 C CNN
+F 2 "" H 5290 960 50  0001 C CNN
+F 3 "" H 5290 960 50  0001 C CNN
+	1    5290 960
+	-1   0    0    1
+$EndComp
+NoConn ~ 2935 1680
+NoConn ~ 5135 4230
+NoConn ~ 5135 4330
+NoConn ~ 5135 4430
+NoConn ~ 5135 4530
+NoConn ~ 5135 4630
+NoConn ~ 5135 4730
+NoConn ~ 4185 5130
+NoConn ~ 2935 4180
+NoConn ~ 2935 4280
+NoConn ~ 2935 4430
+NoConn ~ 2935 4530
+NoConn ~ 2935 4630
+NoConn ~ 2935 4730
+NoConn ~ 2935 4830
+Wire Wire Line
+	5135 1880 5830 1880
+$Comp
+L Device:Jumper_NC_Dual JP1
+U 1 1 60E4CAF5
+P 5290 860
+F 0 "JP1" H 5290 1099 50  0000 C CNN
+F 1 "Jumper_3.3V" H 5290 1008 50  0000 C CNN
+F 2 "Connector_PinSocket_2.54mm:PinSocket_1x03_P2.54mm_Vertical" H 5290 860 50  0001 C CNN
+F 3 "~" H 5290 860 50  0001 C CNN
+	1    5290 860
+	1    0    0    -1
+$EndComp
 Wire Wire Line
 	4780 860  5040 860
-$Comp
-L Device:Jumper_NC_Dual JP?
-U 1 1 60E4CAF5
-P 5381 910
-F 0 "JP?" H 5381 1149 50  0000 C CNN
-F 1 "Jumper_3.3V" H 5381 1058 50  0000 C CNN
-F 2 "" H 5381 910 50  0001 C CNN
-F 3 "~" H 5381 910 50  0001 C CNN
-	1    5381 910
-	1    0    0    -1
-$EndComp
+Wire Wire Line
+	5540 860  5830 860
+Wire Wire Line
+	5830 860  5830 1880
+Wire Wire Line
+	6920 3385 6817 3385
+Wire Wire Line
+	6817 3385 6817 3442
 $EndSCHEMATC

Commit message: test
Parts:
- removed J21: PCB_2, Connector_JST:JST_XH_B6B-XH-A_1x06_P2.50mm_Vertical, symbol Connector:Screw_Terminal_01x06
- removed J23: Ser1, Connector_JST:JST_XH_B5B-XH-A_1x05_P2.50mm_Vertical, symbol Connector:Screw_Terminal_01x05
- removed U1: DOIT-ESP32-DEVKIT-V1, teensy_library-master:ESP32-DOIT-DEVKIT, symbol Ardumower-rescue:DOIT-ESP32-DEVKIT-V1-doit-esp32-devkit-v1
- added J1: ODO_Left, Connector_JST:JST_XH_B4B-XH-A_1x04_P2.50mm_Vertical, symbol Connector:Screw_Terminal_01x04
- added J11: Cutter, Connector_JST:JST_XH_B5B-XH-A_1x05_P2.50mm_Vertical, symbol Connector:Screw_Terminal_01x05
- added J16: Power_Board, Connector_JST:JST_XH_B6B-XH-A_1x06_P2.50mm_Vertical, symbol Connector:Screw_Terminal_01x06
- added J6: ODO_Right, Connector_JST:JST_XH_B4B-XH-A_1x04_P2.50mm_Vertical, symbol Connector:Screw_Terminal_01x04
- added J7: Motor_Right1, Connector_JST:JST_XH_B5B-XH-A_1x05_P2.50mm_Vertical, symbol Connector:Screw_Terminal_01x05
- added J8: Motor_Left1, Connector_JST:JST_XH_B5B-XH-A_1x05_P2.50mm_Vertical, symbol Connector:Screw_Terminal_01x05
- added JP3: MotorPower, Connector_PinSocket_2.54mm:PinSocket_1x03_P2.54mm_Vertical, symbol Device:Jumper_NC_Dual
- added JP4: Jumper, Connector_PinSocket_2.54mm:PinSocket_1x02_P2.54mm_Vertical, symbol Device:Jumper
- added JP5: CutterPower, Connector_PinSocket_2.54mm:PinSocket_1x03_P2.54mm_Vertical, symbol Device:Jumper_NC_Dual
- added R12, R13: 1,5KO, Resistor_THT:R_Axial_DIN0207_L6.3mm_D2.5mm_P2.54mm_Vertical, symbol Device:R
- added R5, R6: 1KO, Resistor_THT:R_Axial_DIN0207_L6.3mm_D2.5mm_P2.54mm_Vertical, symbol Device:R
- added U1: DOIT-ESP32-DEVKIT-V1, teensy_library-master:ESP32-DOIT-DEVKIT, symbol doit-esp32-devkit-v1:DOIT-ESP32-DEVKIT-V1
- added U2: GY-521, teensy_library-master:GY-521, symbol teensy:GY-521
- H1, H2, H3, H4: footprint MountingHole:MountingHole_2.2mm_M2_Pad_TopBottom -> MountingHole:MountingHole_3.2mm_M3_Pad_TopBottom
- J2: value I2C2 -> I2C2_0
- J3: value I2C0 -> I2C0_0
- J30: value I2C1 -> I2C1_0
- J4: value I2C3 -> I2C1_1
- R1, R3: value XXX -> XXXX
Connections:
- net DUE_3.3V is gone; now on net +3V3: R11.2
- net +3V3: now also R3.1, J1.4 (Pin_4), J16.6 (Pin_6), J6.4 (Pin_4), JP3.3, JP4.2, JP5.3, U2.1 (VCC); no longer R3.2
- net +5V: now also J1.3 (Pin_3), J6.3 (Pin_3), JP3.1, JP5.1, U1.18 (VIN)
- net GND: now also J1.2 (Pin_2), J11.2 (Pin_2), J16.5 (Pin_5), J6.2 (Pin_2), J7.2 (Pin_2), J8.2 (Pin_2), R12.2, R13.2, U1.17 (GND), U2.2 (GND)
- net RX1: now also U1.28 (GPIO17_UART2-TX)
- net SCL0: now also U2.3 (SCL)
- net SCL2: now also J16.3 (Pin_3)
- net SDA0: now also R3.2, U2.4 (SDA); no longer R3.1
- net SDA2: now also J16.4 (Pin_4)
- net TX1: now also U1.27 (GPIO16_UART2-RX)
- net pinBatterySwitch: now also J16.2 (Pin_2)
- net pinChargeEnable: now also J16.1 (Pin_1)
- net pinMotorLeftDir: now also J8.4 (Pin_4)
- net pinMotorLeftEnable: now also J8.5 (Pin_5)
- net pinMotorLeftPWM: now also J8.3 (Pin_3)
- net pinMotorMowDir: now also J11.4 (Pin_4)
- net pinMotorMowEnable: now also J11.5 (Pin_5)
- net pinMotorMowPWM: now also J11.3 (Pin_3)
- net pinMotorRightDir: now also J7.4 (Pin_4)
- net pinMotorRightEnable: now also J7.5 (Pin_5)
- net pinMotorRightPWM: now also J7.3 (Pin_3)
- net pinOdometryLeft: now also R6.2
- net pinOdometryRight: now also R5.2
- new net: JP4.1, U2.7 (AD0)
- new net: J1.1 (Pin_1), R12.1, R5.1
- new net: J6.1 (Pin_1), R13.1, R6.1
- new net: J11.1 (Pin_1), JP5.2
- new net: J7.1 (Pin_1), J8.1 (Pin_1), JP3.2
- no-connect marks 18 -> 21
Other:
- moved on the sheet: D7, J2, J25, J30, J31, J4, R2, R4

Commit message: test
Connections:
- net pinSonarLeftEcho: now also U3.18 (26_A12_MOSI1)
- net pinSonarLeftTrigger: now also U3.20 (28_RX7)
- net pinSonarRightEcho: now also U3.19 (27_A13_SCK1)
- net pinSonarRightTrigger: now also U3.21 (29_TX7)
- net pinBatteryVoltage: no longer names the net of U3.43 (21_A7_RX5_BCLK1)
- net pinChargeCurrent: no longer names the net of U3.32 (40_A16)
- net pinChargeVoltage: no longer names the net of U3.33 (41_A17)
Other:
- moved on the sheet: D2, J1, J14, J31, J6, JP2, JP4, R11, R12, R13, R5, R6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

Commit message: test
Parts:
- removed JP2: Buzzer OFF, Connector_PinSocket_2.54mm:PinSocket_1x02_P2.54mm_Vertical, symbol Jumper:Jumper_2_Open
- added BT1: Battery_Cell, Battery:BatteryHolder_Keystone_103_1x20mm, symbol Device:Battery_Cell
Connections:
- net GND: now also BT1.2 (-)
- net pinBuzzer: now also SP1.2
- net at U3.50 (VBAT): now also BT1.1 (+)
- no-connect marks 21 -> 24
Changed lines of the file:
@@
 	1    0    0    -1
 $EndComp
-Text GLabel 8950 1000 0    50   Input ~ 0
+Text GLabel 9350 1000 0    50   Input ~ 0
 pinBuzzer
 $Comp
@@
 	1    9350 800
 	0    1    1    0
-$EndComp
-$Comp
-L Jumper:Jumper_2_Open JP2
-U 1 1 6093522B
-P 9150 1000
-F 0 "JP2" H 9150 1100 50  0000 C CNN
-F 1 "Buzzer OFF" H 9150 900 50  0000 C CNN
-F 2 "Connector_PinSocket_2.54mm:PinSocket_1x02_P2.54mm_Vertical" H 9150 1000 50  0001 C CNN
-F 3 "~" H 9150 1000 50  0001 C CNN
-	1    9150 1000
-	1    0    0    -1
 $EndComp
 $Comp
@@
 Text GLabel 2935 3580 0    50   Output ~ 0
 pinSonarLeftTrigger
+$Comp
+L Device:Battery_Cell BT1
+U 1 1 60EE371C
+P 3300 5150
+F 0 "BT1" V 3045 5200 50  0000 C CNN
+F 1 "Battery_Cell" V 3136 5200 50  0000 C CNN
+F 2 "Battery:BatteryHolder_Keystone_103_1x20mm" V 3300 5210 50  0001 C CNN
+F 3 "~" V 3300 5210 50  0001 C CNN
+	1    3300 5150
+	0    1    1    0
+$EndComp
+$Comp
+L power:GND #PWR046
+U 1 1 60EE61C7
+P 3200 5150
+F 0 "#PWR046" H 3200 4900 50  0001 C CNN
+F 1 "GND" H 3205 4977 50  0000 C CNN
+F 2 "" H 3200 5150 50  0001 C CNN
+F 3 "" H 3200 5150 50  0001 C CNN
+	1    3200 5150
+	1    0    0    -1
+$EndComp
+Wire Wire Line
+	3500 5150 3735 5150
+Wire Wire Line
+	3735 5118 3735 5130
+Connection ~ 3735 5130
+Wire Wire Line
+	3735 5130 3735 5150
+NoConn ~ 4335 5130
+NoConn ~ 4035 5130
+NoConn ~ 3885 5130
 $EndSCHEMATC

Commit message: teensy pcb
Parts:
- removed JP4: Jumper, Connector_PinSocket_2.54mm:PinSocket_1x02_P2.54mm_Vertical, symbol Device:Jumper
- removed U1: DOIT-ESP32-DEVKIT-V1, teensy_library-master:ESP32-DOIT-DEVKIT, symbol doit-esp32-devkit-v1:DOIT-ESP32-DEVKIT-V1
- added J17: Power_PCB2, Connector_JST:JST_XH_B2B-XH-A_1x02_P2.50mm_Vertical, symbol Connector:Screw_Terminal_01x02
- added J18: Free01_02, Connector_JST:JST_XH_B3B-XH-A_1x03_P2.50mm_Vertical, symbol Connector:Screw_Terminal_01x03
- added J20: Can3, Connector_JST:JST_XH_B5B-XH-A_1x05_P2.50mm_Vertical, symbol Connector:Screw_Terminal_01x05
- added J21: Ser5, Connector_JST:JST_XH_B5B-XH-A_1x05_P2.50mm_Vertical, symbol Connector:Screw_Terminal_01x05
- added J22: FreeA16_A17, Connector_JST:JST_XH_B4B-XH-A_1x04_P2.50mm_Vertical, symbol Connector:Screw_Terminal_01x04
- added J23: ESP RFID1, Connector_JST:JST_XH_B5B-XH-A_1x05_P2.50mm_Vertical, symbol Connector:Screw_Terminal_01x05
- added J24: ESP RFID2, Connector_JST:JST_XH_B5B-XH-A_1x05_P2.50mm_Vertical, symbol Connector:Screw_Terminal_01x05
- added J26: ESP32 I2C, Connector_JST:JST_XH_B4B-XH-A_1x04_P2.50mm_Vertical, symbol Connector:Screw_Terminal_01x04
- added R14, R15: XXX, Resistor_THT:R_Axial_DIN0207_L6.3mm_D2.5mm_P2.54mm_Vertical, symbol Device:R
- added U4: ESP32-DEVKIT-V1, teensy_library-master:ESP32-DEVKIT-V1, symbol teensy:ESP32-DEVKIT-V1
- J16: value Power_Board -> Power_PCB1
Connections:
- net +3V3: now also J20.2 (Pin_2), J21.2 (Pin_2), J22.1 (Pin_1)
- net +5V: now also J20.1 (Pin_1), J21.1 (Pin_1), J23.2 (Pin_2), U4.15 (VIN)
- net GND: now also J18.1 (Pin_1), J20.3 (Pin_3), J21.3 (Pin_3), J22.2 (Pin_2), J23.1 (Pin_1), J26.1 (Pin_1), U4.14 (GND)
- net RX1: now also U4.22 (TX2)
- net SCL0: now also J16.3 (Pin_3)
- net SCL1: now also J16.1 (Pin_1)
- net SCL2: no longer J16.3 (Pin_3)
- net SDA0: now also J16.4 (Pin_4)
- net SDA1: now also J16.2 (Pin_2)
- net SDA2: no longer J16.4 (Pin_4)
- net TX1: now also U4.21 (RX2)
- net pinBatterySwitch: now also J17.2 (Pin_2); no longer J16.2 (Pin_2)
- net pinChargeEnable: now also J17.1 (Pin_1); no longer J16.1 (Pin_1)
- net CRX3: now reaches U3.22 (30_CRX3)
- net CRX3: now also J20.5 (Pin_5)
- net CTX3: now reaches U3.23 (31_CTX3)
- net CTX3: now also J20.4 (Pin_4)
- net Free02: now reaches U3.24 (32_OUT1B)
- net Free02: now also J18.3 (Pin_3)
- net FreeA16: now reaches U3.32 (40_A16)
- net FreeA16: now also J22.3 (Pin_3)
- net FreeA17: now reaches U3.33 (41_A17)
- net FreeA17: now also J22.4 (Pin_4)
- net Free01: now reaches U3.35 (13_SCK_LED)
- net Free01: now also J18.2 (Pin_2)
- net TX5: now reaches U3.42 (20_A6_TX5_LRCLK1)
- net TX5: now also J21.4 (Pin_4)
- net RX5: now reaches U3.43 (21_A7_RX5_BCLK1)
- net RX5: now also J21.5 (Pin_5)
- new net: J23.5 (Pin_5), U4.11 (GPIO14_ADC2-CH6_HSPI-CLK_RTC-GPIO16)
- new net: J23.4 (Pin_4), U4.12 (GPIO12_ADC2-CH5_HSPI-MISO_RTC-GPIO15)
- new net: J23.3 (Pin_3), U4.13 (GPIO13_ADC2-CH4_HSPI-MOSI_RTC-GPIO14)
- new net: J24.4 (Pin_4), J26.4 (Pin_4), R14.1, R15.1, U4.16 (3V3)
- new net: J26.2 (Pin_2), R14.2, U4.18 (GPIO15_ADC2-CH3_HSPI-CS0_RTC-GPIO13)
- new net: J26.3 (Pin_3), R15.2, U4.20 (GPIO4_ADC2-CH0_RTC-GPIO10)
- new net: J24.3 (Pin_3), U4.24 (GPIO18_VSPI-CLK)
- new net: J24.2 (Pin_2), U4.25 (GPIO19_VSPI-MISO)
- new net: J24.1 (Pin_1), U4.30 (GPIO23_VSPI-MOSI)
- no-connect marks 24 -> 28
Other:
- moved on the sheet: J11, J14, J31, J7, J8, JP3, JP5, SP1

Commit message: ordered teensy pcb
Parts:
- added J27: ESP32 Sens1, Connector_JST:JST_XH_B3B-XH-A_1x03_P2.50mm_Vertical, symbol Connector:Screw_Terminal_01x03
- added J28: ESP32 FREE, Connector_JST:JST_XH_B4B-XH-A_1x04_P2.50mm_Vertical, symbol Connector:Screw_Terminal_01x04
- added J32: ESP32 Sens2, Connector_JST:JST_XH_B3B-XH-A_1x03_P2.50mm_Vertical, symbol Connector:Screw_Terminal_01x03
- added J33: ESP32 I2C/SER, Connector_JST:JST_XH_B4B-XH-A_1x04_P2.50mm_Vertical, symbol Connector:Screw_Terminal_01x04
- added J34: Teensy On/Off, Connector_JST:JST_XH_B2B-XH-A_1x02_P2.50mm_Vertical, symbol Connector:Screw_Terminal_01x02
- added R16, R17: 1.5KO, Resistor_THT:R_Axial_DIN0207_L6.3mm_D2.5mm_P2.54mm_Vertical, symbol Device:R
- added R18, R19: 1KO, Resistor_THT:R_Axial_DIN0207_L6.3mm_D2.5mm_P2.54mm_Vertical, symbol Device:R
Connections:
- net +5V: now also J27.1 (Pin_1), J32.1 (Pin_1)
- net GND: now also J27.2 (Pin_2), J32.2 (Pin_2), R16.2, R17.2
- net at U3.52 (GND): now also J34.2 (Pin_2)
- net at U3.54 (ON_OFF): now also J34.1 (Pin_1)
- net at U4.26 (GPIO21_I2C-SDA): now also J33.3 (Pin_3)
- net at U4.27 (GPIO3__UART0-RX): now also J33.2 (Pin_2)
- net at U4.28 (GPIO1_UART0-TX): now also J33.1 (Pin_1)
- net at U4.29 (GPIO22_I2C-SCL): now also J33.4 (Pin_4)
- net at U4.4 (GPIO34_ADC1-CH6_RTC-GPIO4): now also R18.2
- net at U4.5 (GPIO35_ADC1-CH7_RTC-GPIO5): now also R19.2
- net at U4.6 (GPIO32_ADC1-CH4_RTC-GPIO9): now also J28.4 (Pin_4)
- net at U4.7 (GPIO33_ADC1-CH5_RTC-GPIO8): now also J28.3 (Pin_3)
- net at U4.8 (GPIO25_ADC2-CH8_DAC1_RTC-GPIO6): now also J28.2 (Pin_2)
- net at U4.9 (GPIO26_ADC2-CH9_DAC2_RTC-GPIO7): now also J28.1 (Pin_1)
- new net: J27.3 (Pin_3), R16.1, R18.1
- new net: J32.3 (Pin_3), R17.1, R19.1
- no-connect marks 28 -> 32
