File: PCB/Power_PCB_v106/charge_pcb.sch (KiCad schematic (older format))
At the start: 48 parts, among them J1 Main_PCB2, J10 Mot_Left, J11 DC/DC1, J12 DC/DC2, J2 Battery, J3 Power Switch, J4 Mow3, J5 Main_PCB1, J6 Mow2, J7 Mow1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

Commit message: teensy_pcb
Parts:
- D3: value 1N4148 -> NOT USE
- R10, R11: value 2k2 -> 4k7
Changed lines of the file:
@@
 P 4800 2350
 F 0 "D3" V 4754 2430 50  0000 L CNN
-F 1 "1N4148" V 4845 2430 50  0000 L CNN
+F 1 "NOT USE" V 4845 2430 50  0000 L CNN
 F 2 "Diode_THT:D_DO-35_SOD27_P7.62mm_Horizontal" H 4800 2175 50  0001 C CNN
 F 3 "https://assets.nexperia.com/documents/data-sheet/1N4148_1N4448.pdf" H 4800 2350 50  0001 C CNN
@@
 P 7275 2435
 F 0 "R10" V 7482 2435 50  0000 C CNN
-F 1 "2k2" V 7391 2435 50  0000 C CNN
+F 1 "4k7" V 7391 2435 50  0000 C CNN
 F 2 "Resistor_THT:R_Axial_DIN0207_L6.3mm_D2.5mm_P7.62mm_Horizontal" V 7205 2435 50  0001 C CNN
 F 3 "~" H 7275 2435 50  0001 C CNN
@@
 P 2615 2250
 F 0 "R11" V 2822 2250 50  0000 C CNN
-F 1 "2k2" V 2731 2250 50  0000 C CNN
+F 1 "4k7" V 2731 2250 50  0000 C CNN
 F 2 "Resistor_THT:R_Axial_DIN0207_L6.3mm_D2.5mm_P7.62mm_Horizontal" V 2545 2250 50  0001 C CNN
 F 3 "~" H 2615 2250 50  0001 C CNN
